File: hardware/New_Multirotor_CPU_imu_V1.3.brd (EAGLE design)
At the start: 50 x 50 mm, 88 parts, among them X2 telemetry, X3 programm, X4 sonar

Commit message: Fixed a bug with baro
удалил версию 1.2 добавил 1.3...
Parts:
- renumbered JP2 to BOOT0, LED6 to LED1-6, SV1 to SPI, SV2 to UART_GPS, TP3 to SWDIO, TP4 to SWCLK, X2 to TELEMETRY, X3 to PROG, X4 to SONAR
Connections:
- net GND: now also DD5.4, DD5.5; no longer DD5.2
- net VCC: now also DD5.2; no longer DD5.4, DD5.5
Routing:
- net GND: track 123.2 -> 129.7 mm
- net VCC: track 198.5 -> 195.7 mm, vias 8 -> 7
- net RADIO_1: track 10.3 -> 9.59 mm
Other:
- board text added: "ADC1"
- board text added: "ADC2"
- board text added: "ADC3"
- board text added: "ADC4"
- board text added: "GPIO1"
- board text added: "GPIO2"
- board text added: "MULTIROTORCONTROL"
- board text added: "S1"
- board text added: "S2"
- board text added: "S3"
- board text added: "S4"
- board text added: "STM32F407VGT6"
- board text added: "V1.2"
