File: hardware/New_Multirotor_CPU_imu_V1.3.sch (EAGLE design)
At the start: 88 parts, among them X2 telemetry, X3 programm, X4 sonar

Commit message: Fixed a bug with baro
удалил версию 1.2 добавил 1.3...
Parts:
- renumbered JP2 to BOOT0, LED6 to LED1-6, SV1 to SPI, SV2 to UART_GPS, TP3 to SWDIO, TP4 to SWCLK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
Connections:
- net GND: now also DD5.CS, DD5.CS1; no longer DD5.PS
- net VCC: now also DD5.PS; no longer DD5.CS, DD5.CS1
